File: kicadFiles/mad-hatter.sch (KiCad schematic (older format))
At the start: 155 parts, among them J1 USB_B_Mini, J2 AVR-ISP-6, U1 ATMEGA32U4, X1 16MHz

Commit message: Placed RGB LEDs
Parts:
- removed C1, C2: 22p, Capacitor_SMD:C_0805_2012Metric_Pad1.15x1.40mm_HandSolder, symbol passives:C_nonpol
- removed C3, C4, C5, C6: 0.1u, Capacitor_SMD:C_0805_2012Metric_Pad1.15x1.40mm_HandSolder, symbol passives:C_nonpol
- removed C7: 4.7u, Capacitor_SMD:C_0805_2012Metric_Pad1.15x1.40mm_HandSolder, symbol passives:C_nonpol
- removed C8: 1u, Capacitor_SMD:C_0805_2012Metric_Pad1.15x1.40mm_HandSolder, symbol passives:C_nonpol
- removed D_0, D_1, D_2, D_3, D_4, D_5, D_6, D_7, D_8, D_9, D_A1, D_ALT1, D_ALT2, D_B1, D_B2, D_BACKSPACE1, D_BSLSH1, D_BSLSH2, D_C1, D_CAPS_LOCK1, D_COMMA1, D_CTRL1, D_CTRL2, D_D1, D_DOT1, D_E1, D_ENTER1, D_EQUAL1, D_F1, D_FN1, D_G1, D_GUI1, D_H1, D_I1, D_J1, D_K1, D_L1, D_M1, D_MINUS1, D_N1, D_O1, D_P1, D_PGDN1, D_PGUP1, D_PRSCR1, D_Q1, D_QUOTE1, D_R1, D_S1, D_SEMIC1, D_SHIFT1, D_SHIFT2, D_SLASH1, D_SPC1, D_SPC2, D_T1, D_TAB1, D_U1, D_V1, D_W1, D_X1, D_Y1, D_Z1, D_[1, D_]1, D_`1: D, acheronComponents:D_SOD-123, symbol Device:D
- removed F1: 1A, Fuse:Fuse_1206_3216Metric_Pad1.42x1.75mm_HandSolder, symbol Device:Polyfuse_Small
- removed J2: AVR-ISP-6, keyboard_parts:AVR_ICSP_3x2, symbol Connector:AVR-ISP-6
- removed K_0, K_1, K_2, K_3, K_4, K_5, K_6, K_7, K_8, K_9, K_A1, K_ALT1, K_ALT2, K_B1, K_B2, K_BACKSPACE1, K_BACKSPACE2, K_BSLSH1, K_BSLSH2, K_C1, K_CAPS_LOCK1, K_CAPS_LOCK1_2, K_COMMA1, K_CTRL1, K_CTRL2, K_D1, K_DOT1, K_E1, K_ENTER1, K_EQUAL1, K_F1, K_FN1, K_G1, K_GUI1, K_GUI1_2, K_H1, K_I1, K_J1, K_K1, K_L1, K_M1, K_MINUS1, K_N1, K_O1, K_P1, K_PGDN1, K_PGUP1, K_PRSCR1, K_Q1, K_QUOTE1, K_R1, K_S1, K_SEMIC1, K_SHIFT1, K_SHIFT2, K_SHIFT2_2, K_SLASH1, K_SPC1, K_SPC1_2, K_SPC2, K_T1, K_TAB1, K_U1, K_V1, K_W1, K_X1, K_Y1, K_Z1, K_[1, K_]1, K_`1: KEYSW, acheronKeyboardSwitches:MX100H, symbol keyboard_parts:KEYSW
- removed R1, R4: 10k, Resistor_SMD:R_0805_2012Metric_Pad1.15x1.40mm_HandSolder, symbol keyboard_parts:R
- removed R2, R3: 22, Resistor_SMD:R_0805_2012Metric_Pad1.15x1.40mm_HandSolder, symbol keyboard_parts:R
- removed RSW1: SW_PUSH, acheronHardware:smdPushBtn, symbol keyboard_parts:SW_PUSH
- removed U1: ATMEGA32U4, keyboard_parts:QFP44_reflow, symbol keyboard_parts:ATMEGA32U4
- removed X1: 16MHz, Crystal:Crystal_SMD_3225-4Pin_3.2x2.5mm, symbol Device:Crystal_GND24
- added D1, D10, D11, D12, D13, D14, D15, D16, D17, D18, D19, D2, D20, D21, D22, D23, D24, D25, D26, D27, D28, D29, D3, D30, D31, D32, D33, D34, D35, D36, D37, D38, D39, D4, D40, D41, D42, D43, D44, D45, D46, D47, D48, D49, D5, D50, D51, D52, D53, D54, D55, D56, D57, D58, D59, D6, D60, D61, D62, D63, D64, D7, D8, D9: SK6812MINI-E, Acheron Components:SK6812MINI_3535_6028_3.2x2.8mm_Round, symbol acheronSymbols:SK6812MINI-E
- added G1: MountingHole, Mad Hatter Graphics:mad_hatter_logo-20x22, symbol Mechanical:MountingHole
- added L1: L_Core_Ferrite, Inductor_SMD:L_1206_3216Metric_Pad1.42x1.75mm_HandSolder, symbol Device:L_Core_Ferrite
- added LED1, LED2, LED3: LED, Acheron Components:LED_THT_2.54mm, symbol acheronSymbols:LED
- added SW1: ESC, Acheron MX SolderMask:MX100, symbol acheronSymbols:MXSwitch
- added SW10: 8, Acheron MX SolderMask:MX100, symbol acheronSymbols:MXSwitch
- added SW11: 9, Acheron MX SolderMask:MX100, symbol acheronSymbols:MXSwitch
- added SW12: 0, Acheron MX SolderMask:MX100, symbol acheronSymbols:MXSwitch
- added SW13: MINUS, Acheron MX SolderMask:MX100, symbol acheronSymbols:MXSwitch
- added SW14: EQUAL, Acheron MX SolderMask:MX100, symbol acheronSymbols:MXSwitch
- added SW15: 2U BKSP, Acheron MX SolderMask:MX200, symbol acheronSymbols:MXSwitch
- added SW16: PGUP, Acheron MX SolderMask:MX100, symbol acheronSymbols:MXSwitch
- added SW17: TAB, Acheron MX SolderMask:MX150, symbol acheronSymbols:MXSwitch
- added SW18: Q, Acheron MX SolderMask:MX100, symbol acheronSymbols:MXSwitch
- added SW19: W, Acheron MX SolderMask:MX100, symbol acheronSymbols:MXSwitch
- added SW2: GRV, Acheron MX SolderMask:MX100, symbol acheronSymbols:MXSwitch
- added SW20: E, Acheron MX SolderMask:MX100, symbol acheronSymbols:MXSwitch
- added SW21: R, Acheron MX SolderMask:MX100, symbol acheronSymbols:MXSwitch
- added SW22: T, Acheron MX SolderMask:MX100, symbol acheronSymbols:MXSwitch
- added SW23: Y, Acheron MX SolderMask:MX100, symbol acheronSymbols:MXSwitch
- added SW24: U, Acheron MX SolderMask:MX100, symbol acheronSymbols:MXSwitch
- added SW25: I, Acheron MX SolderMask:MX100, symbol acheronSymbols:MXSwitch
- added SW26: O, Acheron MX SolderMask:MX100, symbol acheronSymbols:MXSwitch
- added SW27: P, Acheron MX SolderMask:MX100, symbol acheronSymbols:MXSwitch
- added SW28: LBRACE, Acheron MX SolderMask:MX100, symbol acheronSymbols:MXSwitch
- added SW29: RBRACE, Acheron MX SolderMask:MX100, symbol acheronSymbols:MXSwitch
- added SW3: 1, Acheron MX SolderMask:MX100, symbol acheronSymbols:MXSwitch
- added SW30: BACK SLASH, Acheron MX SolderMask:MX150, symbol acheronSymbols:MXSwitch
- added SW31: PGDN, Acheron MX SolderMask:MX100, symbol acheronSymbols:MXSwitch
- added SW32: FULL CAPS, Acheron MX SolderMask:MX175, symbol acheronSymbols:MXSwitch
- added SW33: A, Acheron MX SolderMask:MX100, symbol acheronSymbols:MXSwitch
- added SW34: S, Acheron MX SolderMask:MX100, symbol acheronSymbols:MXSwitch
- added SW35: D, Acheron MX SolderMask:MX100, symbol acheronSymbols:MXSwitch
- added SW36: F, Acheron MX SolderMask:MX100, symbol acheronSymbols:MXSwitch
- added SW37: G, Acheron MX SolderMask:MX100, symbol acheronSymbols:MXSwitch
- added SW38: H, Acheron MX SolderMask:MX100, symbol acheronSymbols:MXSwitch
- added SW39: J, Acheron MX SolderMask:MX100, symbol acheronSymbols:MXSwitch
- added SW4: 2, Acheron MX SolderMask:MX100, symbol acheronSymbols:MXSwitch
- added SW40: K, Acheron MX SolderMask:MX100, symbol acheronSymbols:MXSwitch
- added SW41: L, Acheron MX SolderMask:MX100, symbol acheronSymbols:MXSwitch
- added SW42: COLON, Acheron MX SolderMask:MX100, symbol acheronSymbols:MXSwitch
- added SW43: QUOTE, Acheron MX SolderMask:MX100, symbol acheronSymbols:MXSwitch
- added SW44: ENTER, Acheron MX SolderMask:MX225R, symbol acheronSymbols:MXSwitch
- added SW45: LSHIFT, Acheron MX SolderMask:MX225, symbol acheronSymbols:MXSwitch
- added SW46: Z, Acheron MX SolderMask:MX100, symbol acheronSymbols:MXSwitch
- added SW47: X, Acheron MX SolderMask:MX100, symbol acheronSymbols:MXSwitch
- added SW48: C, Acheron MX SolderMask:MX100, symbol acheronSymbols:MXSwitch
- added SW49: V, Acheron MX SolderMask:MX100, symbol acheronSymbols:MXSwitch
- added SW5: 3, Acheron MX SolderMask:MX100, symbol acheronSymbols:MXSwitch
- added SW50: B, Acheron MX SolderMask:MX100, symbol acheronSymbols:MXSwitch
- added SW51: EXTRA, Acheron MX SolderMask:MX100, symbol acheronSymbols:MXSwitch
- added SW52: N, Acheron MX SolderMask:MX100, symbol acheronSymbols:MXSwitch
- added SW53: M, Acheron MX SolderMask:MX100, symbol acheronSymbols:MXSwitch
- added SW54: COMMA, Acheron MX SolderMask:MX100, symbol acheronSymbols:MXSwitch
- added SW55: DOT, Acheron MX SolderMask:MX100, symbol acheronSymbols:MXSwitch
- added SW56: SLASH, Acheron MX SolderMask:MX100, symbol acheronSymbols:MXSwitch
- added SW57: 2.75U RSHIFT, Acheron MX SolderMask:MX275, symbol acheronSymbols:MXSwitch
- added SW58: LCTRL, Acheron MX SolderMask:MX150, symbol acheronSymbols:MXSwitch
- added SW59: LALT, Acheron MX SolderMask:MX150, symbol acheronSymbols:MXSwitch
- added SW6: 4, Acheron MX SolderMask:MX100, symbol acheronSymbols:MXSwitch
- added SW60: LEFT SPACE, Acheron MX SolderMask:MX200R, symbol acheronSymbols:MXSwitch
- added SW61: LEFT SPACE, Acheron MX SolderMask:MX125, symbol acheronSymbols:MXSwitch
- added SW62: RIGHT SPACE, Acheron MX SolderMask:MX275R, symbol acheronSymbols:MXSwitch
- added SW63: RIGHT ALT, Acheron MX SolderMask:MX150, symbol acheronSymbols:MXSwitch
- added SW64: RIGHT CTRL, Acheron MX SolderMask:MX150, symbol acheronSymbols:MXSwitch
- added SW7: 5, Acheron MX SolderMask:MX100, symbol acheronSymbols:MXSwitch
- added SW8: 6, Acheron MX SolderMask:MX100, symbol acheronSymbols:MXSwitch
- added SW9: 7, Acheron MX SolderMask:MX100, symbol acheronSymbols:MXSwitch
- J1: footprint acheronConnectors:miniB_connector -> Acheron Connectors:USB_MiniB_XM7D-0512
Connections:
- net GND: now also L1.1, LED1.K, LED2.K, LED3.K; no longer J1.5 (GND)
- net GNDPWR: now reaches J1.6 (Shield)
- net GNDPWR: now also J1.5 (GND), L1.2
- net VCC: no longer names the net of J1.1 (VBUS)
- no-connect marks 5 -> 0

Commit message: Further developments
- Placed some capacitors for the RGBs
- Introduced rotary encoders
- Added indicator LEDs resistors
- Rounded corners of the PCB
Parts:
- added C1, C10, C11, C12, C13, C14, C15, C2, C3, C31, C32, C33, C34, C35, C36, C37, C38, C39, C4, C40, C41, C42, C43, C44, C45, C5, C59, C6, C60, C61, C62, C63, C64, C7, C8, C9: 100n, Acheron Components:C_0805_2012Metric_Pad1.15x1.40mm_HandSolder_UP, symbol Device:C_Small
- added C16, C17, C18, C19, C20, C21, C22, C23, C24, C25, C26, C27, C28, C29, C30, C46, C47, C48, C49, C50, C51, C52, C53, C54, C55, C56, C57: 100n, mad_hatter_components:C_0805_2012Metric_Pad1.15x1.40mm_HandSolder_DOWN, symbol Device:C_Small
- added C58: 100n, Capacitor_SMD:C_0805_2012Metric_Pad1.15x1.40mm_HandSolder, symbol Device:C_Small
- added D1, D10, D11, D12, D13, D14, D15, D16, D17, D18, D19, D2, D20, D21, D22, D23, D24, D25, D26, D27, D28, D29, D3, D30, D31, D32, D33, D34, D35, D36, D37, D38, D39, D4, D40, D41, D42, D43, D44, D45, D46, D47, D48, D49, D5, D50, D51, D52, D53, D54, D55, D56, D57, D58, D59, D6, D60, D61, D62, D63, D64, D7, D8, D9: 1N4148W, Acheron Components:D_SOD-123, symbol Device:D
- added R1, R2, R3: 420R, Acheron Components:R_SMD_1206, symbol Device:R_Small
- added R10, R11, R12, R13, R14, R15, R16, R17, R18, R19, R20, R21, R22, R23, R24, R25, R26, R27, R28, R29, R30, R31, R32, R33, R34, R35, R36, R37, R38, R39, R4, R40, R41, R42, R43, R44, R45, R46, R47, R48, R49, R5, R50, R51, R52, R53, R54, R55, R56, R57, R58, R59, R6, R60, R61, R62, R63, R64, R65, R66, R67, R7, R8, R9: 3R, Resistor_SMD:R_1206_3216Metric_Pad1.42x1.75mm_HandSolder, symbol Device:R_Small
- added SW65, SW66, SW67: Rotary_Encoder_Switch_Chassis, Acheron Hardware:ALPS_EC11E, symbol acheronSymbols:Rotary_Encoder_Switch_Chassis
- added U1: USBLC6-2SC6, Acheron Components:SOT-23-6, symbol Power_Protection:USBLC6-2SC6
- D109: renamed from D45; footprint Acheron Components:SK6812MINI_3535_6028_3.2x2.8mm_Round -> mad_hatter_components:SK6812MINI_3535_6028_3.2x2.8mm_Round_DOWN
- D110: renamed from D46; footprint Acheron Components:SK6812MINI_3535_6028_3.2x2.8mm_Round -> mad_hatter_components:SK6812MINI_3535_6028_3.2x2.8mm_Round_DOWN
- D111: renamed from D47; footprint Acheron Components:SK6812MINI_3535_6028_3.2x2.8mm_Round -> mad_hatter_components:SK6812MINI_3535_6028_3.2x2.8mm_Round_DOWN
- D112: renamed from D48; footprint Acheron Components:SK6812MINI_3535_6028_3.2x2.8mm_Round -> mad_hatter_components:SK6812MINI_3535_6028_3.2x2.8mm_Round_DOWN
- D113: renamed from D49; footprint Acheron Components:SK6812MINI_3535_6028_3.2x2.8mm_Round -> mad_hatter_components:SK6812MINI_3535_6028_3.2x2.8mm_Round_DOWN
- D114: renamed from D50; footprint Acheron Components:SK6812MINI_3535_6028_3.2x2.8mm_Round -> mad_hatter_components:SK6812MINI_3535_6028_3.2x2.8mm_Round_DOWN
- D115: renamed from D51; footprint Acheron Components:SK6812MINI_3535_6028_3.2x2.8mm_Round -> mad_hatter_components:SK6812MINI_3535_6028_3.2x2.8mm_Round_DOWN
- D116: renamed from D52; footprint Acheron Components:SK6812MINI_3535_6028_3.2x2.8mm_Round -> mad_hatter_components:SK6812MINI_3535_6028_3.2x2.8mm_Round_DOWN
- D117: renamed from D53; footprint Acheron Components:SK6812MINI_3535_6028_3.2x2.8mm_Round -> mad_hatter_components:SK6812MINI_3535_6028_3.2x2.8mm_Round_DOWN
- D118: renamed from D54; footprint Acheron Components:SK6812MINI_3535_6028_3.2x2.8mm_Round -> mad_hatter_components:SK6812MINI_3535_6028_3.2x2.8mm_Round_DOWN
- D119: renamed from D55; footprint Acheron Components:SK6812MINI_3535_6028_3.2x2.8mm_Round -> mad_hatter_components:SK6812MINI_3535_6028_3.2x2.8mm_Round_DOWN
- D120: renamed from D56; footprint Acheron Components:SK6812MINI_3535_6028_3.2x2.8mm_Round -> mad_hatter_components:SK6812MINI_3535_6028_3.2x2.8mm_Round_DOWN
- D121: renamed from D57; footprint Acheron Components:SK6812MINI_3535_6028_3.2x2.8mm_Round -> mad_hatter_components:SK6812MINI_3535_6028_3.2x2.8mm_Round_DOWN
- D80: renamed from D16; footprint Acheron Components:SK6812MINI_3535_6028_3.2x2.8mm_Round -> mad_hatter_components:SK6812MINI_3535_6028_3.2x2.8mm_Round_DOWN
- D81: renamed from D17; footprint Acheron Components:SK6812MINI_3535_6028_3.2x2.8mm_Round -> mad_hatter_components:SK6812MINI_3535_6028_3.2x2.8mm_Round_DOWN
- D82: renamed from D18; footprint Acheron Components:SK6812MINI_3535_6028_3.2x2.8mm_Round -> mad_hatter_components:SK6812MINI_3535_6028_3.2x2.8mm_Round_DOWN
- D83: renamed from D19; footprint Acheron Components:SK6812MINI_3535_6028_3.2x2.8mm_Round -> mad_hatter_components:SK6812MINI_3535_6028_3.2x2.8mm_Round_DOWN
- D84: renamed from D20; footprint Acheron Components:SK6812MINI_3535_6028_3.2x2.8mm_Round -> mad_hatter_components:SK6812MINI_3535_6028_3.2x2.8mm_Round_DOWN
- D85: renamed from D21; footprint Acheron Components:SK6812MINI_3535_6028_3.2x2.8mm_Round -> mad_hatter_components:SK6812MINI_3535_6028_3.2x2.8mm_Round_DOWN
- D86: renamed from D22; footprint Acheron Components:SK6812MINI_3535_6028_3.2x2.8mm_Round -> mad_hatter_components:SK6812MINI_3535_6028_3.2x2.8mm_Round_DOWN
- D87: renamed from D23; footprint Acheron Components:SK6812MINI_3535_6028_3.2x2.8mm_Round -> mad_hatter_components:SK6812MINI_3535_6028_3.2x2.8mm_Round_DOWN
- D88: renamed from D24; footprint Acheron Components:SK6812MINI_3535_6028_3.2x2.8mm_Round -> mad_hatter_components:SK6812MINI_3535_6028_3.2x2.8mm_Round_DOWN
- D89: renamed from D25; footprint Acheron Components:SK6812MINI_3535_6028_3.2x2.8mm_Round -> mad_hatter_components:SK6812MINI_3535_6028_3.2x2.8mm_Round_DOWN
- D90: renamed from D26; footprint Acheron Components:SK6812MINI_3535_6028_3.2x2.8mm_Round -> mad_hatter_components:SK6812MINI_3535_6028_3.2x2.8mm_Round_DOWN
- D91: renamed from D27; footprint Acheron Components:SK6812MINI_3535_6028_3.2x2.8mm_Round -> mad_hatter_components:SK6812MINI_3535_6028_3.2x2.8mm_Round_DOWN
- D92: renamed from D28; footprint Acheron Components:SK6812MINI_3535_6028_3.2x2.8mm_Round -> mad_hatter_components:SK6812MINI_3535_6028_3.2x2.8mm_Round_DOWN
- D93: renamed from D29; footprint Acheron Components:SK6812MINI_3535_6028_3.2x2.8mm_Round -> mad_hatter_components:SK6812MINI_3535_6028_3.2x2.8mm_Round_DOWN
- D94: renamed from D30; footprint Acheron Components:SK6812MINI_3535_6028_3.2x2.8mm_Round -> mad_hatter_components:SK6812MINI_3535_6028_3.2x2.8mm_Round_DOWN
- J1: value USB_B_Mini -> U-M-M5DD-W-1; footprint Acheron Connectors:USB_MiniB_XM7D-0512 -> Acheron Connectors:U-M-M5DD-W-1; LCSC Part No (none) -> C145778; Manufacturer (none) -> Korean Hroparts Elec; Manufacturer Part No (none) -> U-M-M5DD-W-1
- L1: value L_Core_Ferrite -> 120R@100MHz; LCSC Part No (none) -> C127313; Manufacturer (none) -> TAITEC; Manufacturer Part No (none) -> HCB3216KF-101T30; Package (none) -> L1206
- renumbered D36 to D100, D37 to D101, D38 to D102, D39 to D103, D40 to D104, D41 to D105, D42 to D106, D43 to D107, D44 to D108, D58 to D122, D59 to D123, D60 to D124, D61 to D125, D62 to D126, D63 to D127, D64 to D128, D1 to D65, D2 to D66, D3 to D67, D4 to D68, D5 to D69, D6 to D70, D7 to D71, D8 to D72, D9 to D73, D10 to D74, D11 to D75, D12 to D76, D13 to D77, D14 to D78, D15 to D79, D31 to D95, D32 to D96, D33 to D97, D34 to D98, D35 to D99
Connections:
- net GND: now also D100.3 (VSS), D101.3 (VSS), D102.3 (VSS), D103.3 (VSS), D104.3 (VSS), D105.3 (VSS), D106.3 (VSS), D107.3 (VSS), D108.3 (VSS), D109.3 (VSS), D110.3 (VSS), D111.3 (VSS), D112.3 (VSS), D113.3 (VSS), D114.3 (VSS), D115.3 (VSS), D116.3 (VSS), D117.3 (VSS), D118.3 (VSS), D119.3 (VSS), D120.3 (VSS), D121.3 (VSS), D122.3 (VSS), D123.3 (VSS), D124.3 (VSS), D125.3 (VSS), D126.3 (VSS), D127.3 (VSS), D128.3 (VSS), D65.3 (VSS), D66.3 (VSS), D67.3 (VSS), D68.3 (VSS), D69.3 (VSS), D70.3 (VSS), D71.3 (VSS), D72.3 (VSS), D73.3 (VSS), D74.3 (VSS), D75.3 (VSS), D76.3 (VSS), D77.3 (VSS), D78.3 (VSS), D79.3 (VSS), D80.3 (VSS), D81.3 (VSS), D82.3 (VSS), D83.3 (VSS), D84.3 (VSS), D85.3 (VSS), D86.3 (VSS), D87.3 (VSS), D88.3 (VSS), D89.3 (VSS), D90.3 (VSS), D91.3 (VSS), D92.3 (VSS), D93.3 (VSS), D94.3 (VSS), D95.3 (VSS), D96.3 (VSS), D97.3 (VSS), D98.3 (VSS), D99.3 (VSS), C1.1, C10.1, C11.1, C12.1, C13.1, C14.1, C15.1, C16.1, C17.1, C18.1, C19.1, C2.1, C20.1, C21.1, C22.1, C23.1, C24.1, C25.1, C26.1, C27.1, C28.1, C29.1, C3.1, C30.1, C31.1, C32.1, C33.1, C34.1, C35.1, C36.1, C37.1, C38.1, C39.1, C4.1, C40.1, C41.1, C42.1, C43.1, C44.1, C45.1, C46.1, C47.1, C48.1, C49.1, C5.1, C50.1, C51.1, C52.1, C53.1, C54.1, C55.1, C56.1, C57.1, C58.1, C59.1, C6.1, C60.1, C61.1, C62.1, C63.1, C64.1, C7.1, C8.1, C9.1
- net GNDPWR: now also U1.2 (GND)
- net COL2: now reaches SW2.1 (Col)
- net COL2: now also SW17.1 (Col), SW32.1 (Col), SW45.1 (Col), SW58.1 (Col)
- net at SW2.2 (Row): now also D2.2 (A)
- net COL3: now reaches SW3.1 (Col)
- net COL3: now also SW18.1 (Col), SW33.1 (Col), SW46.1 (Col)
- net at SW3.2 (Row): now also D3.2 (A)
- net COL4: now reaches SW4.1 (Col)
- net COL4: now also SW19.1 (Col), SW34.1 (Col), SW47.1 (Col)
- net at SW4.2 (Row): now also D4.2 (A)
- net COL5: now reaches SW5.1 (Col)
- net COL5: now also SW20.1 (Col), SW35.1 (Col), SW48.1 (Col), SW59.1 (Col)
- net at SW5.2 (Row): now also D5.2 (A)
- net COL6: now reaches SW6.1 (Col)
- net COL6: now also SW21.1 (Col), SW36.1 (Col), SW49.1 (Col), SW60.1 (Col)
- net at SW6.2 (Row): now also D6.2 (A)
- net COL7: now reaches SW7.1 (Col)
- net COL7: now also SW22.1 (Col), SW37.1 (Col), SW50.1 (Col), SW61.1 (Col)
- net at SW7.2 (Row): now also D7.2 (A)
- net COL8: now reaches SW8.1 (Col)
- net COL8: now also SW23.1 (Col), SW38.1 (Col), SW51.1 (Col), SW62.1 (Col)
- net at SW8.2 (Row): now also D8.2 (A)
- net COL1: now reaches SW1.1 (Col)
- net COL1: now also SW16.1 (Col), SW31.1 (Col)
- net at SW1.2 (Row): now also D1.2 (A)
- net VBUS: now reaches J1.1 (VBUS)
- net VBUS: now also U1.5 (VBUS)
- net DBUS-: now reaches J1.2 (D-)
- net DBUS-: now also U1.4 (IO2)
- net DBUS+: now reaches J1.3 (D+)
- net DBUS+: now also U1.6 (IO1)
- net COL9: now reaches SW9.1 (Col)
- net COL9: now also SW24.1 (Col), SW39.1 (Col), SW52.1 (Col), SW63.1 (Col)
- net at SW9.2 (Row): now also D9.2 (A)
- net COL10: now reaches SW10.1 (Col)
- net COL10: now also SW25.1 (Col), SW40.1 (Col), SW53.1 (Col)
- net at SW10.2 (Row): now also D10.2 (A)
- net COL11: now reaches SW11.1 (Col)
- net COL11: now also SW26.1 (Col), SW41.1 (Col), SW54.1 (Col), SW64.1 (Col)
- net at SW11.2 (Row): now also D11.2 (A)
- net COL12: now reaches SW12.1 (Col)
- net COL12: now also SW27.1 (Col), SW42.1 (Col), SW55.1 (Col)
- net at SW12.2 (Row): now also D12.2 (A)
- net COL13: now reaches SW13.1 (Col)
- net COL13: now also SW28.1 (Col), SW43.1 (Col), SW56.1 (Col)
- net at SW13.2 (Row): now also D13.2 (A)
- net COL14: now reaches SW14.1 (Col)
- net COL14: now also SW29.1 (Col), SW57.1 (Col)
- net at SW14.2 (Row): now also D14.2 (A)
- net COL15: now reaches SW15.1 (Col)
- net COL15: now also SW30.1 (Col), SW44.1 (Col)
- net at SW15.2 (Row): now also D15.2 (A)
- net at D65.1 (VDD): now also C1.2, R4.2
- net at SW22.2 (Row): now also D22.2 (A)
- net at SW27.2 (Row): now also D27.2 (A)
- net at SW19.2 (Row): now also D19.2 (A)
- net at SW16.2 (Row): now also D16.2 (A)
- net at SW21.2 (Row): now also D21.2 (A)
- net at SW20.2 (Row): now also D20.2 (A)
- net at SW28.2 (Row): now also D28.2 (A)
- net at SW24.2 (Row): now also D24.2 (A)
- net at SW18.2 (Row): now also D18.2 (A)
- net at SW23.2 (Row): now also D23.2 (A)
- net at SW17.2 (Row): now also D17.2 (A)
- net at SW25.2 (Row): now also D25.2 (A)
- net at SW30.2 (Row): now also D30.2 (A)
- net at SW29.2 (Row): now also D29.2 (A)
- net at SW26.2 (Row): now also D26.2 (A)
- net at D66.1 (VDD): now also C2.2, R5.2
- net at D67.1 (VDD): now also C3.2, R6.2
- net at D68.1 (VDD): now also C4.2, R7.2
- net at D70.1 (VDD): now also C6.2, R9.2
- net at D69.1 (VDD): now also C5.2, R8.2
- net at D71.1 (VDD): now also C7.2, R10.2
- net at D72.1 (VDD): now also C8.2, R11.2
- net at SW33.2 (Row): now also D33.2 (A)
- net at SW41.2 (Row): now also D41.2 (A)
- net at SW32.2 (Row): now also D32.2 (A)
- net at SW40.2 (Row): now also D40.2 (A)
- net at SW37.2 (Row): now also D37.2 (A)
- net at SW36.2 (Row): now also D36.2 (A)
- net at SW38.2 (Row): now also D38.2 (A)
- net at SW35.2 (Row): now also D35.2 (A)
- net at SW43.2 (Row): now also D43.2 (A)
- net at SW42.2 (Row): now also D42.2 (A)
- net at SW34.2 (Row): now also D34.2 (A)
- net at SW44.2 (Row): now also D44.2 (A)
- net at SW31.2 (Row): now also D31.2 (A)
- net at SW39.2 (Row): now also D39.2 (A)
- net at D73.1 (VDD): now also C9.2, R12.2
- net at D74.1 (VDD): now also C10.2, R13.2
- net at D75.1 (VDD): now also C11.2, R14.2
- net at D78.1 (VDD): now also C14.2, R17.2
- net at D77.1 (VDD): now also C13.2, R16.2
- net at D76.1 (VDD): now also C12.2, R15.2
- net at D79.1 (VDD): now also C15.2, R18.2
- net at SW51.2 (Row): now also D51.2 (A)
- net at SW47.2 (Row): now also D47.2 (A)
- net at SW50.2 (Row): now also D50.2 (A)
- net at SW53.2 (Row): now also D53.2 (A)
- net at SW54.2 (Row): now also D54.2 (A)
- net at SW49.2 (Row): now also D49.2 (A)
- net at SW45.2 (Row): now also D45.2 (A)
- net at SW48.2 (Row): now also D48.2 (A)
- net at SW52.2 (Row): now also D52.2 (A)
- net at SW46.2 (Row): now also D46.2 (A)
- net at SW55.2 (Row): now also D55.2 (A)
- net at D80.1 (VDD): now also C16.2, R19.2
- net at SW56.2 (Row): now also D56.2 (A)
- net at SW57.2 (Row): now also D57.2 (A)
- net at D89.1 (VDD): now also C25.2, R28.2
- net at D94.1 (VDD): now also C30.2, R33.2
- net at D88.1 (VDD): now also C24.2, R27.2
- net at D91.1 (VDD): now also C27.2, R30.2
- net at D93.1 (VDD): now also C29.2, R32.2
- net at D90.1 (VDD): now also C26.2, R29.2
- net at D92.1 (VDD): now also C28.2, R31.2
- net at D83.1 (VDD): now also C19.2, R22.2
- net at D86.1 (VDD): now also C22.2, R25.2
- net at D84.1 (VDD): now also C20.2, R23.2
- net at D81.1 (VDD): now also C17.2, R20.2
- net at D82.1 (VDD): now also C18.2, R21.2
- net at D85.1 (VDD): now also C21.2, R24.2
- net at D87.1 (VDD): now also C23.2, R26.2
- net at SW58.2 (Row): now also D58.2 (A)
- net at SW59.2 (Row): now also D59.2 (A)
- net at SW60.2 (Row): now also D60.2 (A)
- net at SW61.2 (Row): now also D61.2 (A)
- net at SW62.2 (Row): now also D62.2 (A)
- net at SW63.2 (Row): now also D63.2 (A)
- net at D101.1 (VDD): now also C37.2, R40.2
- net at D107.1 (VDD): now also C43.2, R46.2
- net at D95.1 (VDD): now also C31.2, R34.2
- net at D100.1 (VDD): now also C36.2, R39.2
- net at D106.1 (VDD): now also C42.2, R45.2
- net at D99.1 (VDD): now also C35.2, R38.2
- net at D109.1 (VDD): now also C45.2, R48.2
- net at D104.1 (VDD): now also C40.2, R43.2
- net at D105.1 (VDD): now also C41.2, R44.2
- net at D98.1 (VDD): now also C34.2, R37.2
- net at D103.1 (VDD): now also C39.2, R42.2
- net at D108.1 (VDD): now also C44.2, R47.2
- net at D96.1 (VDD): now also C32.2, R35.2
- net at D102.1 (VDD): now also C38.2, R41.2
- net at D97.1 (VDD): now also C33.2, R36.2
- net at SW64.2 (Row): now also D64.2 (A)
- net at LED1.A: now also R1.1
- net at LED2.A: now also R2.1
- net at LED3.A: now also R3.1
- net at D122.1 (VDD): now also C58.2, R61.2
- net at D124.1 (VDD): now also C60.2, R63.2
- net at D117.1 (VDD): now also C53.2, R56.2
- net at D110.1 (VDD): now also C46.2, R49.2
- net at D113.1 (VDD): now also C49.2, R52.2
- net at D118.1 (VDD): now also C54.2, R57.2
- net at D116.1 (VDD): now also C52.2, R55.2
- net at D119.1 (VDD): now also C55.2, R58.2
- net at D123.1 (VDD): now also C59.2, R62.2
- net at D115.1 (VDD): now also C51.2, R54.2
- net at D120.1 (VDD): now also C56.2, R59.2
- net at D111.1 (VDD): now also C47.2, R50.2
- net at D114.1 (VDD): now also C50.2, R53.2
- net at D121.1 (VDD): now also C57.2, R60.2
- net at D112.1 (VDD): now also C48.2, R51.2
- net at D125.1 (VDD): now also C61.2, R64.2
- net at D127.1 (VDD): now also C63.2, R66.2
- net at D128.1 (VDD): now also C64.2, R67.2
- net at D126.1 (VDD): now also C62.2, R65.2
- new net 5V: R10.1, R11.1, R12.1, R13.1, R14.1, R15.1, R16.1, R17.1, R18.1, R19.1, R20.1, R21.1, R22.1, R23.1, R24.1, R25.1, R26.1, R27.1, R28.1, R29.1, R30.1, R31.1, R32.1, R33.1, R34.1, R35.1, R36.1, R37.1, R38.1, R39.1, R4.1, R40.1, R41.1, R42.1, R43.1, R44.1, R45.1, R46.1, R47.1, R48.1, R49.1, R5.1, R50.1, R51.1, R52.1, R53.1, R54.1, R55.1, R56.1, R57.1, R58.1, R59.1, R6.1, R60.1, R61.1, R62.1, R63.1, R64.1, R65.1, R66.1, R67.1, R7.1, R8.1, R9.1
- new net D+: U1.1 (IO1)
- new net D-: U1.3 (IO2)
- new net INDICATOR1: R1.2
- new net INDICATOR2: R2.2
- new net INDICATOR3: R3.2
- new net ROW1: D1.1 (K), D10.1 (K), D11.1 (K), D12.1 (K), D13.1 (K), D14.1 (K), D15.1 (K), D2.1 (K), D3.1 (K), D4.1 (K), D5.1 (K), D6.1 (K), D7.1 (K), D8.1 (K), D9.1 (K)
- new net ROW2: D16.1 (K), D17.1 (K), D18.1 (K), D19.1 (K), D20.1 (K), D21.1 (K), D22.1 (K), D23.1 (K), D24.1 (K), D25.1 (K), D26.1 (K), D27.1 (K), D28.1 (K), D29.1 (K), D30.1 (K)
- new net ROW3: D31.1 (K), D32.1 (K), D33.1 (K), D34.1 (K), D35.1 (K), D36.1 (K), D37.1 (K), D38.1 (K), D39.1 (K), D40.1 (K), D41.1 (K), D42.1 (K), D43.1 (K), D44.1 (K)
- new net ROW4: D45.1 (K), D46.1 (K), D47.1 (K), D48.1 (K), D49.1 (K), D50.1 (K), D51.1 (K), D52.1 (K), D53.1 (K), D54.1 (K), D55.1 (K), D56.1 (K), D57.1 (K)
- new net ROW5: D58.1 (K), D59.1 (K), D60.1 (K), D61.1 (K), D62.1 (K), D63.1 (K), D64.1 (K)
- no-connect marks 0 -> 1
Other:
- note added: "RGB LEDs"
- note added: "Switch matrix"
- moved on the sheet: D100, D101, D102, D103, D104, D105, D106, D107, D108, D109, D110, D111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
